Commit message: Start with arm_controller package

File: robot_description/urdf/arm.xacro (robot description, xacro)
@@ -53,4 +53,11 @@
             <axis xyz="1 0 0" />
         </joint>
+        <link name="arm_${index}_eef">
+        </link>
+        <joint name="arm_${index}_3_arm_${index}_eef_joint" type="fixed">
+            <parent link="arm_${index}_3" />
+            <child link="arm_${index}_eef" />
+            <origin xyz="0.0 0 -1" rpy="0.0 0.0 0.0" />
+        </joint>
     </xacro:macro>
 </robot>

Commit message: Separate and rename arm controller classes, split velocity controllers

File: robot_description/urdf/arm.xacro (robot description, xacro)
@@ -7,6 +7,6 @@
         <color rgba="0.5 0.5 1 1" />
     </material>
-    <xacro:macro name="arm" params="index y_offset">
-        <link name="arm_${index}_1">
+    <xacro:macro name="arm" params="name y_offset">
+        <link name="${name}_1">
             <visual>
                 <origin xyz="0.0 0.0 -0.5" rpy="0.0 0.0 0.0" />
@@ -17,11 +17,11 @@
             </visual>
         </link>
-        <joint name="base_arm_${index}_1_joint" type="continuous">
+        <joint name="base_${name}_1_joint" type="continuous">
             <parent link="base" />
-            <child link="arm_${index}_1" />
+            <child link="${name}_1" />
             <origin xyz="0.0 ${y_offset} 1.5" rpy="0.0 0.0 0.0" />
             <axis xyz="0 1 0" />
         </joint>
-        <link name="arm_${index}_2">
+        <link name="${name}_2">
             <visual>
                 <origin xyz="0.0 0.0 -0.25" rpy="0.0 0.0 0.0" />
@@ -32,11 +32,11 @@
             </visual>
         </link>
-        <joint name="arm_${index}_1_arm_${index}_2_joint" type="continuous">
-            <parent link="arm_${index}_1" />
-            <child link="arm_${index}_2" />
+        <joint name="${name}_1_${name}_2_joint" type="continuous">
+            <parent link="${name}_1" />
+            <child link="${name}_2" />
             <origin xyz="0.0 0 -1" rpy="0.0 0.0 0.0" />
             <axis xyz="0 0 1" />
         </joint>
-        <link name="arm_${index}_3">
+        <link name="${name}_3">
             <visual>
                 <origin xyz="0.0 0.0 -0.5" rpy="0.0 0.0 0.0" />
@@ -47,15 +47,15 @@
             </visual>
         </link>
-        <joint name="arm_${index}_2_arm_${index}_3_joint" type="continuous">
-            <parent link="arm_${index}_2" />
-            <child link="arm_${index}_3" />
+        <joint name="${name}_2_${name}_3_joint" type="continuous">
+            <parent link="${name}_2" />
+            <child link="${name}_3" />
             <origin xyz="0.0 0 -0.5" rpy="0.0 0.0 0.0" />
             <axis xyz="1 0 0" />
         </joint>
-        <link name="arm_${index}_eef">
+        <link name="${name}_eef">
         </link>
-        <joint name="arm_${index}_3_arm_${index}_eef_joint" type="fixed">
-            <parent link="arm_${index}_3" />
-            <child link="arm_${index}_eef" />
+        <joint name="${name}_3_${name}_eef_joint" type="fixed">
+            <parent link="${name}_3" />
+            <child link="${name}_eef" />
             <origin xyz="0.0 0 -1" rpy="0.0 0.0 0.0" />
         </joint>

File: robot_description/urdf/robot.urdf.xacro (robot description, xacro)
@@ -14,6 +14,6 @@
     </joint>
     <xacro:base />
-    <xacro:arm index="1" y_offset="1.125" />
-    <xacro:arm index="2" y_offset="-1.125" />
+    <xacro:arm name="left_arm" y_offset="1.125" />
+    <xacro:arm name="right_arm" y_offset="-1.125" />
     <xacro:wheel index="1" parent_link="base" y_offset="1.125" z_offset="-1.75" />
     <xacro:wheel index="2" parent_link="base" y_offset="-1.125" z_offset="-1.75" />

File: robot_description/urdf/ros2_control.xacro (robot description, xacro)
@@ -7,30 +7,30 @@
         <param name="calculate_dynamics">true</param>
       </hardware>
-      <joint name="base_arm_1_1_joint">
+      <joint name="base_left_arm_1_joint">
         <command_interface name="velocity" />
         <state_interface name="position" />
         <state_interface name="velocity" />
       </joint>
-      <joint name="arm_1_1_arm_1_2_joint">
+      <joint name="left_arm_1_left_arm_2_joint">
         <command_interface name="velocity" />
         <state_interface name="position" />
         <state_interface name="velocity" />
       </joint>
-      <joint name="arm_1_2_arm_1_3_joint">
+      <joint name="left_arm_2_left_arm_3_joint">
         <command_interface name="velocity" />
         <state_interface name="position" />
         <state_interface name="velocity" />
       </joint>
-      <joint name="base_arm_2_1_joint">
+      <joint name="base_right_arm_1_joint">
         <command_interface name="velocity" />
         <state_interface name="position" />
         <state_interface name="velocity" />
       </joint>
-      <joint name="arm_2_1_arm_2_2_joint">
+      <joint name="right_arm_1_right_arm_2_joint">
         <command_interface name="velocity" />
         <state_interface name="position" />
         <state_interface name="velocity" />
       </joint>
-      <joint name="arm_2_2_arm_2_3_joint">
+      <joint name="right_arm_2_right_arm_3_joint">
         <command_interface name="velocity" />
         <state_interface name="position" />

Commit message: Change arms' third rotation axis from x to y

File: robot_description/urdf/arm.xacro (robot description, xacro)
@@ -51,5 +51,5 @@
             <child link="${name}_3" />
             <origin xyz="0.0 0 -0.5" rpy="0.0 0.0 0.0" />
-            <axis xyz="1 0 0" />
+            <axis xyz="0 1 0" />
         </joint>
         <link name="${name}_eef">
