Commit message: Add tf publisher to base controller

File: robot_description/urdf/base.xacro (robot description, xacro)
@@ -14,8 +14,14 @@
             </visual>
         </link>
-        <joint name="odom_base_joint" type="fixed">
+        <link name="base_wrapper" />
+        <joint name="base_wrapper_base_joint" type="fixed">
             <origin xyz="0.0 0.0 2.25" rpy="0.0 0.0 0" />
+            <parent link="base_wrapper" />
+            <child link="base" />
+        </joint>
+        <joint name="odom_base_wrapper_joint" type="fixed">
+            <origin xyz="0.0 0.0 0.0" rpy="0.0 0.0 0" />
             <parent link="odom" />
-            <child link="base" />
+            <child link="base_wrapper" />
         </joint>
     </xacro:macro>

File: robot_description/urdf/robot.urdf.xacro (robot description, xacro)
@@ -6,5 +6,7 @@
     <xacro:include filename="$(find robot_description)/urdf/ros2_control.xacro" />
     <xacro:wheeled_humanoid_ros2_control />
+    <!-- map -> odom: Localization corrections (ex. SLAM) -->
     <link name="map" />
+    <!-- odom -> base: Robot motion relative to starting position -->
     <link name="odom" />
     <joint name="map_odom_joint" type="fixed">
