Commit message: Rework base kinematics to use differential drive model and start with MPC controller

File: wheeled_humanoid_ros/urdf/robot.urdf.xacro (robot description, xacro)
@@ -20,5 +20,5 @@
     <xacro:wheel index="1" parent_link="base" y_offset="1.125" z_offset="-1.75" />
     <xacro:wheel index="2" parent_link="base" y_offset="-1.125" z_offset="-1.75" />
-    <link name="wheel_3_base">
+    <!-- <link name="wheel_3_base">
         <visual>
             <origin xyz="0.0 0.0 0.0" rpy="0.0 0.0 0.0" />
@@ -43,4 +43,4 @@
         <axis xyz="0 0 1" />
     </joint>
-    <xacro:wheel index="3" parent_link="wheel_3_steering" y_offset="0" z_offset="0" />
+    <xacro:wheel index="3" parent_link="wheel_3_steering" y_offset="0" z_offset="0" /> -->
 </robot>

File: wheeled_humanoid_ros/urdf/ros2_control.xacro (robot description, xacro)
@@ -47,5 +47,5 @@
         <state_interface name="velocity" />
       </joint>
-      <joint name="wheel_3_base_wheel_3_steering_joint">
+      <!-- <joint name="wheel_3_base_wheel_3_steering_joint">
         <command_interface name="velocity" />
         <state_interface name="position" />
@@ -56,5 +56,5 @@
         <state_interface name="position" />
         <state_interface name="velocity" />
-      </joint>
+      </joint> -->
     </ros2_control>
   </xacro:macro>
