Commit message: Randomize spawned target z-positions and let the robot touch them

File: core_ros/urdf/arm.xacro (robot description, xacro)
@@ -8,5 +8,5 @@
     </material>
     <xacro:macro name="arm" params="name y_offset">
-        <link name="${name}_1">
+        <link name="${name}_arm_1">
             <visual>
                 <origin xyz="0.0 0.0 -0.5" rpy="0.0 0.0 0.0" />
@@ -17,11 +17,11 @@
             </visual>
         </link>
-        <joint name="base_${name}_1_joint" type="continuous">
+        <joint name="base_${name}_arm_1_joint" type="continuous">
             <parent link="base" />
-            <child link="${name}_1" />
+            <child link="${name}_arm_1" />
             <origin xyz="0.0 ${y_offset} 1.5" rpy="0.0 0.0 0.0" />
             <axis xyz="0 1 0" />
         </joint>
-        <link name="${name}_2">
+        <link name="${name}_arm_2">
             <visual>
                 <origin xyz="0.0 0.0 -0.25" rpy="0.0 0.0 0.0" />
@@ -32,11 +32,11 @@
             </visual>
         </link>
-        <joint name="${name}_1_${name}_2_joint" type="continuous">
-            <parent link="${name}_1" />
-            <child link="${name}_2" />
+        <joint name="${name}_arm_1_${name}_arm_2_joint" type="continuous">
+            <parent link="${name}_arm_1" />
+            <child link="${name}_arm_2" />
             <origin xyz="0.0 0 -1" rpy="0.0 0.0 0.0" />
             <axis xyz="0 0 1" />
         </joint>
-        <link name="${name}_3">
+        <link name="${name}_arm_3">
             <visual>
                 <origin xyz="0.0 0.0 -0.5" rpy="0.0 0.0 0.0" />
@@ -47,15 +47,15 @@
             </visual>
         </link>
-        <joint name="${name}_2_${name}_3_joint" type="continuous">
-            <parent link="${name}_2" />
-            <child link="${name}_3" />
+        <joint name="${name}_arm_2_${name}_arm_3_joint" type="continuous">
+            <parent link="${name}_arm_2" />
+            <child link="${name}_arm_3" />
             <origin xyz="0.0 0 -0.5" rpy="0.0 0.0 0.0" />
             <axis xyz="0 1 0" />
         </joint>
-        <link name="${name}_eef">
+        <link name="${name}_arm_eef">
         </link>
-        <joint name="${name}_3_${name}_eef_joint" type="fixed">
-            <parent link="${name}_3" />
-            <child link="${name}_eef" />
+        <joint name="${name}_arm_3_${name}_arm_eef_joint" type="fixed">
+            <parent link="${name}_arm_3" />
+            <child link="${name}_arm_eef" />
             <origin xyz="0.0 0 -1" rpy="0.0 0.0 0.0" />
         </joint>

File: core_ros/urdf/robot.urdf.xacro (robot description, xacro)
@@ -16,31 +16,7 @@
     </joint>
     <xacro:base />
-    <xacro:arm name="left_arm" y_offset="1.125" />
-    <xacro:arm name="right_arm" y_offset="-1.125" />
+    <xacro:arm name="left" y_offset="1.125" />
+    <xacro:arm name="right" y_offset="-1.125" />
     <xacro:wheel index="1" parent_link="base" y_offset="1.125" z_offset="-1.75" />
     <xacro:wheel index="2" parent_link="base" y_offset="-1.125" z_offset="-1.75" />
-    <!-- <link name="wheel_3_base">
-        <visual>
-            <origin xyz="0.0 0.0 0.0" rpy="0.0 0.0 0.0" />
-            <geometry>
-                <box size="1.8 0.2 0.125" />
-            </geometry>
-            <material name="white" />
-        </visual>
-    </link>
-    <joint name="base_wheel_3_base_joint" type="fixed">
-        <parent link="base" />
-        <child link="wheel_3_base" />
-        <origin xyz="0.5 0.0 -1.75" rpy="0.0 0.0 0.0" />
-        <axis xyz="1 0 0" />
-    </joint>
-    <link name="wheel_3_steering">
-    </link>
-    <joint name="wheel_3_base_wheel_3_steering_joint" type="continuous">
-        <parent link="wheel_3_base" />
-        <child link="wheel_3_steering" />
-        <origin xyz="0.9 0 0" rpy="0.0 0.0 0.0" />
-        <axis xyz="0 0 1" />
-    </joint>
-    <xacro:wheel index="3" parent_link="wheel_3_steering" y_offset="0" z_offset="0" /> -->
 </robot>
