Commit message: Add URDF collision and isaac lab mdp files

File: src/core_ros/urdf/arm.xacro (robot description, xacro)
@@ -16,4 +16,10 @@
                 <material name="light-blue" />
             </visual>
+            <collision>
+                <origin xyz="0.0 0.0 -0.5" rpy="0.0 0.0 0.0" />
+                <geometry>
+                    <box size="0.5 0.25 1" />
+                </geometry>
+            </collision>
         </link>
         <joint name="base_${name}_arm_1_joint" type="continuous">
@@ -31,4 +37,10 @@
                 <material name="white" />
             </visual>
+            <collision>
+                <origin xyz="0.0 0.0 -0.25" rpy="0.0 0.0 0.0" />
+                <geometry>
+                    <box size="0.25 0.25 0.5" />
+                </geometry>
+            </collision>
         </link>
         <joint name="${name}_arm_1_${name}_arm_2_joint" type="continuous">
@@ -46,4 +58,10 @@
                 <material name="light-blue" />
             </visual>
+            <collision>
+                <origin xyz="0.0 0.0 -0.5" rpy="0.0 0.0 0.0" />
+                <geometry>
+                    <box size="0.25 0.25 1" />
+                </geometry>
+            </collision>
         </link>
         <joint name="${name}_arm_2_${name}_arm_3_joint" type="continuous">

File: src/core_ros/urdf/base.xacro (robot description, xacro)
@@ -5,4 +5,6 @@
     </material>
     <xacro:macro name="base">
+        <!-- Base wrapper link to get a frame with z=0 -->
+        <link name="base_wrapper" />
         <link name="base">
             <visual>
@@ -13,6 +15,11 @@
                 <material name="blue" />
             </visual>
+            <collision>
+                <origin xyz="0.0 0.0 0.0" rpy="0.0 0.0 0.0" />
+                <geometry>
+                    <box size="0.8 2 3.5" />
+                </geometry>
+            </collision>
         </link>
-        <link name="base_wrapper" />
         <joint name="base_wrapper_base_joint" type="fixed">
             <origin xyz="0.0 0.0 2.25" rpy="0.0 0.0 0" />

File: src/core_ros/urdf/wheel.xacro (robot description, xacro)
@@ -13,4 +13,10 @@
                 <material name="pink"/>
             </visual>
+            <collision>
+                <origin xyz="0.0 0.0 0.0" rpy="1.575 0.0 0.0"/>
+                <geometry>
+                    <cylinder length="0.25" radius="0.5"/>
+                </geometry>
+            </collision>
         </link>
         <joint name="${parent_link}_wheel_${index}_joint" type="continuous">
@@ -21,12 +27,3 @@
         </joint>
     </xacro:macro>
-    <!-- <xacro:macro name="wheel_inertial" params="m x y z oy oz" >
-        <inertial>
-            <origin xyz="0 ${oy} ${oz}" rpy="0.0 0.0 0.0"/>
-            <mass value="${m}"/>
-            <inertia    ixx="${(1/12) * m * (z*z + y*y)}" ixy="0.0" ixz="0.0"
-                        iyy="${(1/12) * m * (x*x + z*z)}" iyz="0.0"
-                        izz="${(1/12) * m * (y*y + x*x)}"/>
-        </inertial>
-    </xacro:macro> -->
 </robot>
