Commit message: Add QT GUI command script, create ROS virtual env to use python package, fix URDF fixed frames

File: src/taser_ros/robot_description/urdf/xacro/base.xacro (robot description, xacro)
@@ -27,9 +27,9 @@
             <child link="base" />
         </joint>
-        <joint name="odom_base_wrapper_joint" type="fixed">
+        <!-- <joint name="odom_base_wrapper_joint" type="fixed">
             <origin xyz="0.0 0.0 0.0" rpy="0.0 0.0 0" />
-            <parent link="odom" />
+            <parent link="map" />
             <child link="base_wrapper" />
-        </joint>
+        </joint> -->
     </xacro:macro>
 </robot>

File: src/taser_ros/robot_description/urdf/xacro/robot.urdf.xacro (robot description, xacro)
@@ -7,12 +7,12 @@
     <xacro:taser_ros2_control />
     <!-- map -> odom - Localization corrections (ex. SLAM) -->
-    <link name="map" />
+    <!-- <link name="map" /> -->
     <!-- odom -> base - Robot motion relative to starting position -->
-    <link name="odom" />
-    <joint name="map_odom_joint" type="fixed">
+    <!-- <link name="odom" /> -->
+    <!-- <joint name="map_odom_joint" type="fixed">
         <origin xyz="0.0 0.0 0.0" rpy="0.0 0.0 0" />
         <parent link="map" />
         <child link="odom" />
-    </joint>
+    </joint> -->
     <xacro:base />
     <xacro:arm name="left" y_offset="1.125" />
