Commit message: Remove arm actions in balance task

File: src/taser_ros/robot_description/urdf/xacro/arm.xacro (robot description, xacro)
@@ -28,4 +28,5 @@
             <origin rpy="0.0 0.0 0.0" xyz="0.0 ${offset_sign}0.2625 0.4" />
             <axis xyz="0 1 0" />
+            <dynamics damping="0.1" friction="0.1" />
         </joint>
         <link name="${side}_arm_1">
@@ -70,4 +71,5 @@
             <origin xyz="0.0 0 -0.3" rpy="0.0 0.0 0.0" />
             <axis xyz="0 0 1" />
+            <dynamics damping="0.1" friction="0.1" />
         </joint>
         <link name="${side}_arm_3">
@@ -91,4 +93,5 @@
             <origin xyz="0.0 0 -0.2" rpy="0.0 0.0 0.0" />
             <axis xyz="0 1 0" />
+            <dynamics damping="0.1" friction="0.1" />
         </joint>
         <link name="${side}_arm_eef">

File: src/taser_ros/robot_description/urdf/xacro/wheel.xacro (robot description, xacro)
@@ -25,4 +25,5 @@
             <origin xyz="0.0 ${offset_sign}0.3 -0.5" rpy="0.0 0.0 0.0" />
             <axis xyz="0 1 0" />
+            <dynamics damping="0.01" friction="0.0" />
         </joint>
     </xacro:macro>
