Commit message: Decrease robot size from 3.5m to 1m

File: src/taser_ros/robot_description/urdf/robot.urdf (robot description, URDF)
Before this commit: robot taser, 14 links, 13 joints
Links:
- removed link map
- removed link odom
- link base: geometry collision box size=0.2 0.5 1; visual box size=0.2 0.5 1
- link left_arm_1: geometry collision box size=0.2 0.1 0.3; visual box size=0.2 0.1 0.3
- link left_arm_2: geometry collision box size=0.1 0.1 0.2; visual box size=0.1 0.1 0.2
- link left_arm_3: geometry collision box size=0.1 0.1 0.3; visual box size=0.1 0.1 0.3
- link right_arm_1: geometry collision box size=0.2 0.1 0.3; visual box size=0.2 0.1 0.3
- link right_arm_2: geometry collision box size=0.1 0.1 0.2; visual box size=0.1 0.1 0.2
- link right_arm_3: geometry collision box size=0.1 0.1 0.3; visual box size=0.1 0.1 0.3
- link wheel_1: geometry collision cylinder length=0.1 radius=0.15; visual cylinder length=0.1 radius=0.15
- link wheel_2: geometry collision cylinder length=0.1 radius=0.15; visual cylinder length=0.1 radius=0.15
Joints:
- removed joint map_odom_joint
- removed joint odom_base_wrapper_joint
- joint base_left_arm_1_joint: origin xyz=0.0 1.125 1.5 rpy=0.0 0.0 0.0 -> xyz=0.0 0.3 0.5 rpy=0.0 0.0 0.0
- joint base_right_arm_1_joint: origin xyz=0.0 -1.125 1.5 rpy=0.0 0.0 0.0 -> xyz=0.0 -0.3 0.5 rpy=0.0 0.0 0.0
- joint base_wheel_1_joint: origin xyz=0.0 1.125 -1.75 rpy=0.0 0.0 0.0 -> xyz=0.0 0.3 -0.5 rpy=0.0 0.0 0.0
- joint base_wheel_2_joint: origin xyz=0.0 -1.125 -1.75 rpy=0.0 0.0 0.0 -> xyz=0.0 -0.3 -0.5 rpy=0.0 0.0 0.0
- joint base_wrapper_base_joint: origin xyz=0.0 0.0 2.25 rpy=0.0 0.0 0 -> xyz=0.0 0.0 0.65 rpy=0.0 0.0 0
- joint left_arm_1_left_arm_2_joint: origin xyz=0.0 0 -1 rpy=0.0 0.0 0.0 -> xyz=0.0 0 -0.3 rpy=0.0 0.0 0.0
- joint left_arm_2_left_arm_3_joint: origin xyz=0.0 0 -0.5 rpy=0.0 0.0 0.0 -> xyz=0.0 0 -0.2 rpy=0.0 0.0 0.0
- joint left_arm_3_left_arm_eef_joint: origin xyz=0.0 0 -1 rpy=0.0 0.0 0.0 -> xyz=0.0 0 -0.3 rpy=0.0 0.0 0.0
- joint right_arm_1_right_arm_2_joint: origin xyz=0.0 0 -1 rpy=0.0 0.0 0.0 -> xyz=0.0 0 -0.3 rpy=0.0 0.0 0.0
- joint right_arm_2_right_arm_3_joint: origin xyz=0.0 0 -0.5 rpy=0.0 0.0 0.0 -> xyz=0.0 0 -0.2 rpy=0.0 0.0 0.0
- joint right_arm_3_right_arm_eef_joint: origin xyz=0.0 0 -1 rpy=0.0 0.0 0.0 -> xyz=0.0 0 -0.3 rpy=0.0 0.0 0.0

File: src/taser_ros/robot_description/urdf/xacro/arm.xacro (robot description, xacro)
@@ -10,14 +10,14 @@
         <link name="${name}_arm_1">
             <visual>
-                <origin xyz="0.0 0.0 -0.5" rpy="0.0 0.0 0.0" />
+                <origin xyz="0.0 0.0 -0.15" rpy="0.0 0.0 0.0" />
                 <geometry>
-                    <box size="0.5 0.25 1" />
+                    <box size="0.2 0.1 0.3" />
                 </geometry>
                 <material name="light-blue" />
             </visual>
             <collision>
-                <origin xyz="0.0 0.0 -0.5" rpy="0.0 0.0 0.0" />
+                <origin xyz="0.0 0.0 -0.15" rpy="0.0 0.0 0.0" />
                 <geometry>
-                    <box size="0.5 0.25 1" />
+                    <box size="0.2 0.1 0.3" />
                 </geometry>
             </collision>
@@ -26,19 +26,19 @@
             <parent link="base" />
             <child link="${name}_arm_1" />
-            <origin xyz="0.0 ${y_offset} 1.5" rpy="0.0 0.0 0.0" />
+            <origin xyz="0.0 ${y_offset} 0.5" rpy="0.0 0.0 0.0" />
             <axis xyz="0 1 0" />
         </joint>
         <link name="${name}_arm_2">
             <visual>
-                <origin xyz="0.0 0.0 -0.25" rpy="0.0 0.0 0.0" />
+                <origin xyz="0.0 0.0 -0.1" rpy="0.0 0.0 0.0" />
                 <geometry>
-                    <box size="0.25 0.25 0.5" />
+                    <box size="0.1 0.1 0.2" />
                 </geometry>
                 <material name="white" />
             </visual>
             <collision>
-                <origin xyz="0.0 0.0 -0.25" rpy="0.0 0.0 0.0" />
+                <origin xyz="0.0 0.0 -0.1" rpy="0.0 0.0 0.0" />
                 <geometry>
-                    <box size="0.25 0.25 0.5" />
+                    <box size="0.1 0.1 0.2" />
                 </geometry>
             </collision>
@@ -47,19 +47,19 @@
             <parent link="${name}_arm_1" />
             <child link="${name}_arm_2" />
-            <origin xyz="0.0 0 -1" rpy="0.0 0.0 0.0" />
+            <origin xyz="0.0 0 -0.3" rpy="0.0 0.0 0.0" />
             <axis xyz="0 0 1" />
         </joint>
         <link name="${name}_arm_3">
             <visual>
-                <origin xyz="0.0 0.0 -0.5" rpy="0.0 0.0 0.0" />
+                <origin xyz="0.0 0.0 -0.15" rpy="0.0 0.0 0.0" />
                 <geometry>
-                    <box size="0.25 0.25 1" />
+                    <box size="0.1 0.1 0.3" />
                 </geometry>
                 <material name="light-blue" />
             </visual>
             <collision>
-                <origin xyz="0.0 0.0 -0.5" rpy="0.0 0.0 0.0" />
+                <origin xyz="0.0 0.0 -0.15" rpy="0.0 0.0 0.0" />
                 <geometry>
-                    <box size="0.25 0.25 1" />
+                    <box size="0.1 0.1 0.3" />
                 </geometry>
             </collision>
@@ -68,5 +68,5 @@
             <parent link="${name}_arm_2" />
             <child link="${name}_arm_3" />
-            <origin xyz="0.0 0 -0.5" rpy="0.0 0.0 0.0" />
+            <origin xyz="0.0 0 -0.2" rpy="0.0 0.0 0.0" />
             <axis xyz="0 1 0" />
         </joint>
@@ -76,5 +76,5 @@
             <parent link="${name}_arm_3" />
             <child link="${name}_arm_eef" />
-            <origin xyz="0.0 0 -1" rpy="0.0 0.0 0.0" />
+            <origin xyz="0.0 0 -0.3" rpy="0.0 0.0 0.0" />
         </joint>
     </xacro:macro>

File: src/taser_ros/robot_description/urdf/xacro/base.xacro (robot description, xacro)
@@ -11,5 +11,5 @@
                 <origin xyz="0.0 0.0 0.0" rpy="0.0 0.0 0.0" />
                 <geometry>
-                    <box size="0.8 2 3.5" />
+                    <box size="0.2 0.5 1" />
                 </geometry>
                 <material name="blue" />
@@ -18,18 +18,13 @@
                 <origin xyz="0.0 0.0 0.0" rpy="0.0 0.0 0.0" />
                 <geometry>
-                    <box size="0.8 2 3.5" />
+                    <box size="0.2 0.5 1" />
                 </geometry>
             </collision>
         </link>
         <joint name="base_wrapper_base_joint" type="fixed">
-            <origin xyz="0.0 0.0 2.25" rpy="0.0 0.0 0" />
+            <origin xyz="0.0 0.0 0.65" rpy="0.0 0.0 0" />
             <parent link="base_wrapper" />
             <child link="base" />
         </joint>
-        <!-- <joint name="odom_base_wrapper_joint" type="fixed">
-            <origin xyz="0.0 0.0 0.0" rpy="0.0 0.0 0" />
-            <parent link="map" />
-            <child link="base_wrapper" />
-        </joint> -->
     </xacro:macro>
 </robot>

File: src/taser_ros/robot_description/urdf/xacro/robot.urdf.xacro (robot description, xacro)
@@ -6,17 +6,8 @@
     <xacro:include filename="$(find taser_ros)/robot_description/urdf/xacro/ros2_control.xacro" />
     <xacro:taser_ros2_control />
-    <!-- map -> odom - Localization corrections (ex. SLAM) -->
-    <!-- <link name="map" /> -->
-    <!-- odom -> base - Robot motion relative to starting position -->
-    <!-- <link name="odom" /> -->
-    <!-- <joint name="map_odom_joint" type="fixed">
-        <origin xyz="0.0 0.0 0.0" rpy="0.0 0.0 0" />
-        <parent link="map" />
-        <child link="odom" />
-    </joint> -->
     <xacro:base />
-    <xacro:arm name="left" y_offset="1.125" />
-    <xacro:arm name="right" y_offset="-1.125" />
-    <xacro:wheel index="1" parent_link="base" y_offset="1.125" z_offset="-1.75" />
-    <xacro:wheel index="2" parent_link="base" y_offset="-1.125" z_offset="-1.75" />
+    <xacro:arm name="left" y_offset="0.3" />
+    <xacro:arm name="right" y_offset="-0.3" />
+    <xacro:wheel index="1" parent_link="base" y_offset="0.3" z_offset="-0.5" />
+    <xacro:wheel index="2" parent_link="base" y_offset="-0.3" z_offset="-0.5" />
 </robot>

File: src/taser_ros/robot_description/urdf/xacro/ros2_control.xacro (robot description, xacro)
@@ -47,14 +47,4 @@
         <state_interface name="velocity" />
       </joint>
-      <!-- <joint name="wheel_3_base_wheel_3_steering_joint">
-        <command_interface name="velocity" />
-        <state_interface name="position" />
-        <state_interface name="velocity" />
-      </joint>
-      <joint name="wheel_3_steering_wheel_3_joint">
-        <command_interface name="velocity" />
-        <state_interface name="position" />
-        <state_interface name="velocity" />
-      </joint> -->
     </ros2_control>
   </xacro:macro>

File: src/taser_ros/robot_description/urdf/xacro/wheel.xacro (robot description, xacro)
@@ -9,5 +9,5 @@
                 <origin xyz="0.0 0.0 0.0" rpy="1.575 0.0 0.0"/>
                 <geometry>
-                    <cylinder length="0.25" radius="0.5"/>
+                    <cylinder length="0.1" radius="0.15"/>
                 </geometry>
                 <material name="pink"/>
@@ -16,5 +16,5 @@
                 <origin xyz="0.0 0.0 0.0" rpy="1.575 0.0 0.0"/>
                 <geometry>
-                    <cylinder length="0.25" radius="0.5"/>
+                    <cylinder length="0.1" radius="0.15"/>
                 </geometry>
             </collision>

Commit message: Add shoulder links to the URDF and rename wheel links

File: src/taser_ros/robot_description/urdf/robot.urdf (robot description, URDF)
Before this commit: robot taser, 12 links, 11 joints
Links:
- removed link wheel_1
- removed link wheel_2
- added link left_arm_shoulder; collision cylinder length=0.025 radius=0.075; visual cylinder length=0.025 radius=0.075
- added link left_wheel; collision cylinder length=0.1 radius=0.15; visual cylinder length=0.1 radius=0.15
- added link right_arm_shoulder; collision cylinder length=0.025 radius=0.075; visual cylinder length=0.025 radius=0.075
- added link right_wheel; collision cylinder length=0.1 radius=0.15; visual cylinder length=0.1 radius=0.15
Joints:
- removed joint base_left_arm_1_joint
- removed joint base_right_arm_1_joint
- removed joint base_wheel_1_joint
- removed joint base_wheel_2_joint
- added joint base_left_arm_shoulder_joint: type continuous, parent base, child left_arm_shoulder, origin xyz=0.0 +0.2625 0.4 rpy=0.0 0.0 0.0, axis 0 1 0
- added joint base_left_wheel_joint: type continuous, parent base, child left_wheel, origin xyz=0.0 +0.3 -0.5 rpy=0.0 0.0 0.0, axis 0 1 0
- added joint base_right_arm_shoulder_joint: type continuous, parent base, child right_arm_shoulder, origin xyz=0.0 -0.2625 0.4 rpy=0.0 0.0 0.0, axis 0 1 0
- added joint base_right_wheel_joint: type continuous, parent base, child right_wheel, origin xyz=0.0 -0.3 -0.5 rpy=0.0 0.0 0.0, axis 0 1 0
- added joint left_arm_shoulder_left_arm_1_joint: type fixed, parent left_arm_shoulder, child left_arm_1, origin xyz=0.0 +0.0625 0.1 rpy=0.0 0.0 0.0, axis 0 1 0
- added joint right_arm_shoulder_right_arm_1_joint: type fixed, parent right_arm_shoulder, child right_arm_1, origin xyz=0.0 -0.0625 0.1 rpy=0.0 0.0 0.0, axis 0 1 0

File: src/taser_ros/robot_description/urdf/xacro/arm.xacro (robot description, xacro)
@@ -7,6 +7,27 @@
         <color rgba="0.5 0.5 1 1" />
     </material>
-    <xacro:macro name="arm" params="name y_offset">
-        <link name="${name}_arm_1">
+    <xacro:macro name="arm" params="side offset_sign">
+        <link name="${side}_arm_shoulder">
+            <visual>
+                <origin rpy="1.57 0.0 0.0" xyz="0.0 0.0 0.0" />
+                <geometry>
+                    <cylinder length="0.025" radius="0.075" />
+                </geometry>
+                <material name="light-blue" />
+            </visual>
+            <collision>
+                <origin rpy="0.0 0.0 0.0" xyz="0.0 0.0 -0.15" />
+                <geometry>
+                    <cylinder length="0.025" radius="0.075" />
+                </geometry>
+            </collision>
+        </link>
+        <joint name="base_${side}_arm_shoulder_joint" type="continuous">
+            <parent link="base" />
+            <child link="${side}_arm_shoulder" />
+            <origin rpy="0.0 0.0 0.0" xyz="0.0 ${offset_sign}0.2625 0.4" />
+            <axis xyz="0 1 0" />
+        </joint>
+        <link name="${side}_arm_1">
             <visual>
                 <origin xyz="0.0 0.0 -0.15" rpy="0.0 0.0 0.0" />
@@ -23,11 +44,11 @@
             </collision>
         </link>
-        <joint name="base_${name}_arm_1_joint" type="continuous">
-            <parent link="base" />
-            <child link="${name}_arm_1" />
-            <origin xyz="0.0 ${y_offset} 0.5" rpy="0.0 0.0 0.0" />
+        <joint name="${side}_arm_shoulder_${side}_arm_1_joint" type="fixed">
+            <parent link="${side}_arm_shoulder" />
+            <child link="${side}_arm_1" />
+            <origin rpy="0.0 0.0 0.0" xyz="0.0 ${offset_sign}0.0625 0.1" />
             <axis xyz="0 1 0" />
         </joint>
-        <link name="${name}_arm_2">
+        <link name="${side}_arm_2">
             <visual>
                 <origin xyz="0.0 0.0 -0.1" rpy="0.0 0.0 0.0" />
@@ -44,11 +65,11 @@
             </collision>
         </link>
-        <joint name="${name}_arm_1_${name}_arm_2_joint" type="continuous">
-            <parent link="${name}_arm_1" />
-            <child link="${name}_arm_2" />
+        <joint name="${side}_arm_1_${side}_arm_2_joint" type="continuous">
+            <parent link="${side}_arm_1" />
+            <child link="${side}_arm_2" />
             <origin xyz="0.0 0 -0.3" rpy="0.0 0.0 0.0" />
             <axis xyz="0 0 1" />
         </joint>
-        <link name="${name}_arm_3">
+        <link name="${side}_arm_3">
             <visual>
                 <origin xyz="0.0 0.0 -0.15" rpy="0.0 0.0 0.0" />
@@ -65,15 +86,15 @@
             </collision>
         </link>
-        <joint name="${name}_arm_2_${name}_arm_3_joint" type="continuous">
-            <parent link="${name}_arm_2" />
-            <child link="${name}_arm_3" />
+        <joint name="${side}_arm_2_${side}_arm_3_joint" type="continuous">
+            <parent link="${side}_arm_2" />
+            <child link="${side}_arm_3" />
             <origin xyz="0.0 0 -0.2" rpy="0.0 0.0 0.0" />
             <axis xyz="0 1 0" />
         </joint>
-        <link name="${name}_arm_eef">
+        <link name="${side}_arm_eef">
         </link>
-        <joint name="${name}_arm_3_${name}_arm_eef_joint" type="fixed">
-            <parent link="${name}_arm_3" />
-            <child link="${name}_arm_eef" />
+        <joint name="${side}_arm_3_${side}_arm_eef_joint" type="fixed">
+            <parent link="${side}_arm_3" />
+            <child link="${side}_arm_eef" />
             <origin xyz="0.0 0 -0.3" rpy="0.0 0.0 0.0" />
         </joint>

File: src/taser_ros/robot_description/urdf/xacro/robot.urdf.xacro (robot description, xacro)
@@ -7,7 +7,7 @@
     <xacro:taser_ros2_control />
     <xacro:base />
-    <xacro:arm name="left" y_offset="0.3" />
-    <xacro:arm name="right" y_offset="-0.3" />
-    <xacro:wheel index="1" parent_link="base" y_offset="0.3" z_offset="-0.5" />
-    <xacro:wheel index="2" parent_link="base" y_offset="-0.3" z_offset="-0.5" />
+    <xacro:arm side="left" offset_sign="+" />
+    <xacro:arm side="right" offset_sign="-" />
+    <xacro:wheel side="left" offset_sign="+" />
+    <xacro:wheel side="right" offset_sign="-" />
 </robot>

File: src/taser_ros/robot_description/urdf/xacro/ros2_control.xacro (robot description, xacro)
@@ -7,5 +7,5 @@
         <param name="calculate_dynamics">true</param>
       </hardware>
-      <joint name="base_left_arm_1_joint">
+      <joint name="base_left_arm_shoulder_joint">
         <command_interface name="velocity" />
         <state_interface name="position" />
@@ -22,5 +22,5 @@
         <state_interface name="velocity" />
       </joint>
-      <joint name="base_right_arm_1_joint">
+      <joint name="base_right_arm_shoulder_joint">
         <command_interface name="velocity" />
         <state_interface name="position" />
@@ -37,10 +37,10 @@
         <state_interface name="velocity" />
       </joint>
-      <joint name="base_wheel_1_joint">
+      <joint name="base_left_wheel_joint">
         <command_interface name="velocity" />
         <state_interface name="position" />
         <state_interface name="velocity" />
       </joint>
-      <joint name="base_wheel_2_joint">
+      <joint name="base_right_wheel_joint">
         <command_interface name="velocity" />
         <state_interface name="position" />

File: src/taser_ros/robot_description/urdf/xacro/wheel.xacro (robot description, xacro)
@@ -2,27 +2,27 @@
 <robot xmlns:xacro="http://www.ros.org/wiki/xacro">
     <material name="pink">
-        <color rgba="0.3 0 0.2 1"/>
+        <color rgba="0.3 0 0.2 1" />
     </material>
-    <xacro:macro name="wheel" params="index y_offset z_offset parent_link">
-        <link name="wheel_${index}">
+    <xacro:macro name="wheel" params="side offset_sign">
+        <link name="${side}_wheel">
             <visual>
-                <origin xyz="0.0 0.0 0.0" rpy="1.575 0.0 0.0"/>
+                <origin xyz="0.0 0.0 0.0" rpy="1.575 0.0 0.0" />
                 <geometry>
-                    <cylinder length="0.1" radius="0.15"/>
+                    <cylinder length="0.1" radius="0.15" />
                 </geometry>
-                <material name="pink"/>
+                <material name="pink" />
             </visual>
             <collision>
-                <origin xyz="0.0 0.0 0.0" rpy="1.575 0.0 0.0"/>
+                <origin xyz="0.0 0.0 0.0" rpy="1.575 0.0 0.0" />
                 <geometry>
-                    <cylinder length="0.1" radius="0.15"/>
+                    <cylinder length="0.1" radius="0.15" />
                 </geometry>
             </collision>
         </link>
-        <joint name="${parent_link}_wheel_${index}_joint" type="continuous">
-            <parent link="${parent_link}"/>
-            <child link="wheel_${index}"/>
-            <origin xyz="0.0 ${y_offset} ${z_offset}" rpy="0.0 0.0 0.0"/>
-            <axis xyz="0 1 0"/>
+        <joint name="base_${side}_wheel_joint" type="continuous">
+            <parent link="base" />
+            <child link="${side}_wheel" />
+            <origin xyz="0.0 ${offset_sign}0.3 -0.5" rpy="0.0 0.0 0.0" />
+            <axis xyz="0 1 0" />
         </joint>
     </xacro:macro>
