Commit message: Remove base_wrapper link, change Pose2D to Pose, fix damping gains, change XFormPrim to Articulation

File: src/taser_ros/robot_description/urdf/taser.urdf (robot description, URDF)
Before this commit: robot taser, 14 links, 13 joints
Links:
- removed link base
- removed link base_wrapper
- added link base_link; collision box size=0.2 0.5 1; visual box size=0.2 0.5 1
Joints:
- removed joint base_left_arm_shoulder_joint
- removed joint base_left_wheel_joint
- removed joint base_right_arm_shoulder_joint
- removed joint base_right_wheel_joint
- removed joint base_wrapper_base_joint
- added joint base_link_left_arm_shoulder_joint: type continuous, parent base_link, child left_arm_shoulder, origin xyz=0.0 +0.2625 0.4 rpy=0.0 0.0 0.0, axis 0 1 0
- added joint base_link_left_wheel_joint: type continuous, parent base_link, child left_wheel, origin xyz=0.0 +0.3 -0.5 rpy=0.0 0.0 0.0, axis 0 1 0
- added joint base_link_right_arm_shoulder_joint: type continuous, parent base_link, child right_arm_shoulder, origin xyz=0.0 -0.2625 0.4 rpy=0.0 0.0 0.0, axis 0 1 0
- added joint base_link_right_wheel_joint: type continuous, parent base_link, child right_wheel, origin xyz=0.0 -0.3 -0.5 rpy=0.0 0.0 0.0, axis 0 1 0

File: src/taser_ros/robot_description/urdf/xacro/arm.xacro (robot description, xacro)
@@ -23,6 +23,6 @@
             </collision>
         </link>
-        <joint name="base_${side}_arm_shoulder_joint" type="continuous">
-            <parent link="base" />
+        <joint name="base_link_${side}_arm_shoulder_joint" type="continuous">
+            <parent link="base_link" />
             <child link="${side}_arm_shoulder" />
             <origin rpy="0.0 0.0 0.0" xyz="0.0 ${offset_sign}0.2625 0.4" />

File: src/taser_ros/robot_description/urdf/xacro/base.xacro (robot description, xacro)
@@ -5,7 +5,5 @@
     </material>
     <xacro:macro name="base">
-        <!-- Base wrapper link to get a frame with z=0 -->
-        <link name="base_wrapper" />
-        <link name="base">
+        <link name="base_link">
             <visual>
                 <origin xyz="0.0 0.0 0.0" rpy="0.0 0.0 0.0" />
@@ -22,9 +20,4 @@
             </collision>
         </link>
-        <joint name="base_wrapper_base_joint" type="fixed">
-            <origin xyz="0.0 0.0 0.65" rpy="0.0 0.0 0" />
-            <parent link="base_wrapper" />
-            <child link="base" />
-        </joint>
     </xacro:macro>
 </robot>

File: src/taser_ros/robot_description/urdf/xacro/ros2_control.xacro (robot description, xacro)
@@ -7,5 +7,5 @@
         <param name="calculate_dynamics">true</param>
       </hardware>
-      <joint name="base_left_arm_shoulder_joint">
+      <joint name="base_link_left_arm_shoulder_joint">
         <command_interface name="velocity" />
         <state_interface name="position" />
@@ -22,5 +22,5 @@
         <state_interface name="velocity" />
       </joint>
-      <joint name="base_right_arm_shoulder_joint">
+      <joint name="base_link_right_arm_shoulder_joint">
         <command_interface name="velocity" />
         <state_interface name="position" />
@@ -37,10 +37,10 @@
         <state_interface name="velocity" />
       </joint>
-      <joint name="base_left_wheel_joint">
+      <joint name="base_link_left_wheel_joint">
         <command_interface name="velocity" />
         <state_interface name="position" />
         <state_interface name="velocity" />
       </joint>
-      <joint name="base_right_wheel_joint">
+      <joint name="base_link_right_wheel_joint">
         <command_interface name="velocity" />
         <state_interface name="position" />

File: src/taser_ros/robot_description/urdf/xacro/wheel.xacro (robot description, xacro)
@@ -20,6 +20,6 @@
             </collision>
         </link>
-        <joint name="base_${side}_wheel_joint" type="continuous">
-            <parent link="base" />
+        <joint name="base_link_${side}_wheel_joint" type="continuous">
+            <parent link="base_link" />
             <child link="${side}_wheel" />
             <origin xyz="0.0 ${offset_sign}0.3 -0.5" rpy="0.0 0.0 0.0" />
