Commit message: Add lock mechanism to the URDF and USD

File: src/taser/common/model/urdf/taser.urdf (robot description, URDF)
Before this commit: robot taser, 13 links, 12 joints
Links:
- added link back_lock; collision box size=0.02 0.3 0.1732; visual box size=0.02 0.3 0.1732
- added link front_lock; collision box size=0.02 0.3 0.1732; visual box size=0.02 0.3 0.1732
Joints:
- added joint base_link_back_lock_joint: type revolute, parent base_link, child back_lock, origin xyz=-0.1 0.0 -0.5 rpy=0.0 0.5236 0.0, axis 0 1 0, limit lower=0.0 upper=2.618 effort=0.0 velocity=0.0
- added joint base_link_front_lock_joint: type revolute, parent base_link, child front_lock, origin xyz=+0.1 0.0 -0.5 rpy=0.0 -0.5236 0.0, axis 0 1 0, limit lower=-2.618 upper=0.0 effort=0.0 velocity=0.0

File: src/taser/common/model/urdf/xacro/base.xacro (robot description, xacro)
@@ -21,3 +21,27 @@
         </link>
     </xacro:macro>
+    <xacro:macro name="lock" params="side offset_sign default_angle lower_limit upper_limit">
+        <link name="${side}_lock">
+            <visual>
+                <origin rpy="0.0 0.0 0.0" xyz="0.0 0.0 -0.0866" />
+                <geometry>
+                    <box size="0.02 0.3 0.1732" />
+                </geometry>
+                <material name="blue" />
+            </visual>
+            <collision>
+                <origin rpy="0.0 0.0 0.0" xyz="0.0 0.0 -0.0866" />
+                <geometry>
+                    <box size="0.02 0.3 0.1732" />
+                </geometry>
+            </collision>
+        </link>
+        <joint name="base_link_${side}_lock_joint" type="revolute">
+            <parent link="base_link" />
+            <child link="${side}_lock" />
+            <origin rpy="0.0 ${default_angle} 0.0" xyz="${offset_sign}0.1 0.0 -0.5" />
+            <axis xyz="0 1 0" />
+            <limit lower="${lower_limit}" upper="${upper_limit}" effort="0.0" velocity="0.0" />
+        </joint>
+    </xacro:macro>
 </robot>

File: src/taser/common/model/urdf/xacro/robot.urdf.xacro (robot description, xacro)
@@ -1,10 +1,12 @@
 <?xml version="1.0"?>
 <robot xmlns:xacro="http://www.ros.org/wiki/xacro" name="taser">
-    <xacro:include filename="$(find taser_ros)/robot_description/urdf/xacro/base.xacro" />
-    <xacro:include filename="$(find taser_ros)/robot_description/urdf/xacro/arm.xacro" />
-    <xacro:include filename="$(find taser_ros)/robot_description/urdf/xacro/wheel.xacro" />
-    <xacro:include filename="$(find taser_ros)/robot_description/urdf/xacro/ros2_control.xacro" />
+    <xacro:include filename="./base.xacro" />
+    <xacro:include filename="./arm.xacro" />
+    <xacro:include filename="./wheel.xacro" />
+    <xacro:include filename="./ros2_control.xacro" />
     <xacro:taser_ros2_control />
     <xacro:base />
+    <xacro:lock side="front" offset_sign="+" default_angle="-0.5236" lower_limit="-2.618" upper_limit="0.0" />
+    <xacro:lock side="back" offset_sign="-" default_angle="0.5236" lower_limit="0.0" upper_limit="2.618" />
     <xacro:arm side="left" offset_sign="+" />
     <xacro:arm side="right" offset_sign="-" />

Commit message: Rework lock mechanism and integrate into locomotion policy, improve TaserJointState

File: src/taser/common/model/urdf/taser.urdf (robot description, URDF)
Before this commit: robot taser, 15 links, 14 joints
Links:
- added link back_lock_support; collision box size=0.15 0.4 0.02; visual box size=0.15 0.4 0.02
- added link front_lock_support; collision box size=0.15 0.4 0.02; visual box size=0.15 0.4 0.02
- link back_lock: geometry collision box size=0.025 0.4 1.0; visual box size=0.025 0.4 1.0
- link front_lock: geometry collision box size=0.025 0.4 1.0; visual box size=0.025 0.4 1.0
Joints:
- added joint back_lock_support_joint: type revolute, parent back_lock, child back_lock_support, origin xyz=-0.025 0.0 -0.48 rpy=0.0 0.0 0.0, axis 0 -1 0, limit lower=-1.57 upper=0.0 effort=0.0 velocity=0.0
- added joint front_lock_support_joint: type revolute, parent front_lock, child front_lock_support, origin xyz=+0.025 0.0 -0.48 rpy=0.0 0.0 0.0, axis 0 +1 0, limit lower=-1.57 upper=0.0 effort=0.0 velocity=0.0
- joint base_link_back_lock_joint: axis 0 1 0 -> 0 0 1; limit lower=0.0 upper=2.618 effort=0.0 velocity=0.0 -> lower=0.0 upper=0.15 effort=0.0 velocity=0.0; origin xyz=-0.1 0.0 -0.5 rpy=0.0 0.5236 0.0 -> xyz=-0.1 0.0 -0.15 rpy=0.0 0.0 0.0; type revolute -> prismatic
- joint base_link_front_lock_joint: axis 0 1 0 -> 0 0 1; limit lower=-2.618 upper=0.0 effort=0.0 velocity=0.0 -> lower=0.0 upper=0.15 effort=0.0 velocity=0.0; origin xyz=+0.1 0.0 -0.5 rpy=0.0 -0.5236 0.0 -> xyz=+0.1 0.0 -0.15 rpy=0.0 0.0 0.0; type revolute -> prismatic

File: src/taser/common/model/urdf/xacro/base.xacro (robot description, xacro)
@@ -21,26 +21,50 @@
         </link>
     </xacro:macro>
-    <xacro:macro name="lock" params="side offset_sign default_angle lower_limit upper_limit">
+    <xacro:macro name="lock" params="side offset_sign">
         <link name="${side}_lock">
             <visual>
-                <origin rpy="0.0 0.0 0.0" xyz="0.0 0.0 -0.0866" />
+                <origin rpy="0.0 0.0 0.0" xyz="${offset_sign}0.0125 0.0 0.0" />
                 <geometry>
-                    <box size="0.02 0.3 0.1732" />
+                    <box size="0.025 0.4 1.0" />
                 </geometry>
                 <material name="blue" />
             </visual>
             <collision>
-                <origin rpy="0.0 0.0 0.0" xyz="0.0 0.0 -0.0866" />
+                <origin rpy="0.0 0.0 0.0" xyz="${offset_sign}0.0125 0.0 0.0" />
                 <geometry>
-                    <box size="0.02 0.3 0.1732" />
+                    <box size="0.025 0.4 1.0" />
                 </geometry>
             </collision>
         </link>
-        <joint name="base_link_${side}_lock_joint" type="revolute">
+        <joint name="base_link_${side}_lock_joint" type="prismatic">
             <parent link="base_link" />
             <child link="${side}_lock" />
-            <origin rpy="0.0 ${default_angle} 0.0" xyz="${offset_sign}0.1 0.0 -0.5" />
-            <axis xyz="0 1 0" />
-            <limit lower="${lower_limit}" upper="${upper_limit}" effort="0.0" velocity="0.0" />
+            <origin rpy="0.0 0.0 0.0" xyz="${offset_sign}0.1 0.0 -0.15" />
+            <axis xyz="0 0 1" />
+            <dynamics damping="0.1" friction="0.1" />
+            <limit effort="0.0" lower="0.0" upper="0.15" velocity="0.0" />
+        </joint>
+        <link name="${side}_lock_support">
+            <visual>
+                <origin rpy="0.0 0.0 0.0" xyz="${offset_sign}0.075 0.0 -0.01" />
+                <geometry>
+                    <box size="0.15 0.4 0.02" />
+                </geometry>
+                <material name="blue" />
+            </visual>
+            <collision>
+                <origin rpy="0.0 0.0 0.0" xyz="${offset_sign}0.075 0.0 -0.01" />
+                <geometry>
+                    <box size="0.15 0.4 0.02" />
+                </geometry>
+            </collision>
+        </link>
+        <joint name="${side}_lock_support_joint" type="revolute">
+            <parent link="${side}_lock" />
+            <child link="${side}_lock_support" />
+            <origin rpy="0.0 0.0 0.0" xyz="${offset_sign}0.025 0.0 -0.48" />
+            <axis xyz="0 ${offset_sign}1 0" />
+            <dynamics damping="0.1" friction="0.1" />
+            <limit effort="0.0" lower="-1.57" upper="0.0" velocity="0.0" />
         </joint>
     </xacro:macro>

File: src/taser/common/model/urdf/xacro/robot.urdf.xacro (robot description, xacro)
@@ -7,6 +7,6 @@
     <xacro:taser_ros2_control />
     <xacro:base />
-    <xacro:lock side="front" offset_sign="+" default_angle="-0.5236" lower_limit="-2.618" upper_limit="0.0" />
-    <xacro:lock side="back" offset_sign="-" default_angle="0.5236" lower_limit="0.0" upper_limit="2.618" />
+    <xacro:lock side="front" offset_sign="+" />
+    <xacro:lock side="back" offset_sign="-" />
     <xacro:arm side="left" offset_sign="+" />
     <xacro:arm side="right" offset_sign="-" />

Commit message: Install curobo, start adapting data collection pipeline from thesis

File: src/taser/common/model/urdf/taser.urdf (robot description, URDF)
Before this commit: robot taser, 17 links, 16 joints
Joints:
- joint base_link_left_arm_shoulder_joint: limit (none) -> lower=-3.1416 upper=3.1416 effort=0.0 velocity=1000.0; type continuous -> revolute
- joint base_link_right_arm_shoulder_joint: limit (none) -> lower=-3.1416 upper=3.1416 effort=0.0 velocity=1000.0; type continuous -> revolute
- joint left_arm_1_left_arm_2_joint: limit (none) -> lower=-3.1416 upper=3.1416 effort=0.0 velocity=1000.0; type continuous -> revolute
- joint left_arm_2_left_arm_3_joint: limit (none) -> lower=-3.1416 upper=3.1416 effort=0.0 velocity=1000.0; type continuous -> revolute
- joint left_arm_shoulder_left_arm_1_joint: axis 0 1 0 -> (none)
- joint right_arm_1_right_arm_2_joint: limit (none) -> lower=-3.1416 upper=3.1416 effort=0.0 velocity=1000.0; type continuous -> revolute
- joint right_arm_2_right_arm_3_joint: limit (none) -> lower=-3.1416 upper=3.1416 effort=0.0 velocity=1000.0; type continuous -> revolute
- joint right_arm_shoulder_right_arm_1_joint: axis 0 1 0 -> (none)

File: src/taser/common/model/urdf/xacro/arm.xacro (robot description, xacro)
@@ -23,5 +23,5 @@
             </collision>
         </link>
-        <joint name="base_link_${side}_arm_shoulder_joint" type="continuous">
+        <joint name="base_link_${side}_arm_shoulder_joint" type="revolute">
             <parent link="base_link" />
             <child link="${side}_arm_shoulder" />
@@ -29,4 +29,5 @@
             <axis xyz="0 1 0" />
             <dynamics damping="0.1" friction="0.1" />
+            <limit effort="0.0" lower="-3.1416" upper="3.1416" velocity="1000.0" />
         </joint>
         <link name="${side}_arm_1">
@@ -49,5 +50,4 @@
             <child link="${side}_arm_1" />
             <origin rpy="0.0 0.0 0.0" xyz="0.0 ${offset_sign}0.0625 0.1" />
-            <axis xyz="0 1 0" />
         </joint>
         <link name="${side}_arm_2">
@@ -66,5 +66,5 @@
             </collision>
         </link>
-        <joint name="${side}_arm_1_${side}_arm_2_joint" type="continuous">
+        <joint name="${side}_arm_1_${side}_arm_2_joint" type="revolute">
             <parent link="${side}_arm_1" />
             <child link="${side}_arm_2" />
@@ -72,4 +72,5 @@
             <axis xyz="0 0 1" />
             <dynamics damping="0.1" friction="0.1" />
+            <limit effort="0.0" lower="-3.1416" upper="3.1416" velocity="1000.0" />
         </joint>
         <link name="${side}_arm_3">
@@ -88,5 +89,5 @@
             </collision>
         </link>
-        <joint name="${side}_arm_2_${side}_arm_3_joint" type="continuous">
+        <joint name="${side}_arm_2_${side}_arm_3_joint" type="revolute">
             <parent link="${side}_arm_2" />
             <child link="${side}_arm_3" />
@@ -94,4 +95,5 @@
             <axis xyz="0 1 0" />
             <dynamics damping="0.1" friction="0.1" />
+            <limit effort="0.0" lower="-3.1416" upper="3.1416" velocity="1000.0" />
         </joint>
         <link name="${side}_arm_eef">

Commit message: Add curobo collision spheres, fix arm joint limits and collisions

File: src/taser/common/model/urdf/taser.urdf (robot description, URDF)
Before this commit: robot taser, 17 links, 16 joints
Joints:
- joint base_link_left_arm_shoulder_joint: limit lower=-3.1416 upper=3.1416 effort=0.0 velocity=1000.0 -> effort=0.0 velocity=1000.0; type revolute -> continuous
- joint base_link_right_arm_shoulder_joint: limit lower=-3.1416 upper=3.1416 effort=0.0 velocity=1000.0 -> effort=0.0 velocity=1000.0; type revolute -> continuous
- joint left_arm_1_left_arm_2_joint: limit lower=-3.1416 upper=3.1416 effort=0.0 velocity=1000.0 -> effort=0.0 velocity=1000.0; type revolute -> continuous
- joint left_arm_2_left_arm_3_joint: limit lower=-3.1416 upper=3.1416 effort=0.0 velocity=1000.0 -> lower=-2.3562 upper=2.3562 effort=0.0 velocity=1000.0
- joint right_arm_1_right_arm_2_joint: limit lower=-3.1416 upper=3.1416 effort=0.0 velocity=1000.0 -> effort=0.0 velocity=1000.0; type revolute -> continuous
- joint right_arm_2_right_arm_3_joint: limit lower=-3.1416 upper=3.1416 effort=0.0 velocity=1000.0 -> lower=-2.3562 upper=2.3562 effort=0.0 velocity=1000.0

File: src/taser/common/model/urdf/xacro/arm.xacro (robot description, xacro)
@@ -17,5 +17,5 @@
             </visual>
             <collision>
-                <origin rpy="0.0 0.0 0.0" xyz="0.0 0.0 -0.15" />
+                <origin rpy="1.57 0.0 0.0" xyz="0.0 0.0 0.0" />
                 <geometry>
                     <cylinder length="0.025" radius="0.075" />
@@ -23,5 +23,5 @@
             </collision>
         </link>
-        <joint name="base_link_${side}_arm_shoulder_joint" type="revolute">
+        <joint name="base_link_${side}_arm_shoulder_joint" type="continuous">
             <parent link="base_link" />
             <child link="${side}_arm_shoulder" />
@@ -29,5 +29,5 @@
             <axis xyz="0 1 0" />
             <dynamics damping="0.1" friction="0.1" />
-            <limit effort="0.0" lower="-3.1416" upper="3.1416" velocity="1000.0" />
+            <limit effort="0.0" velocity="1000.0" />
         </joint>
         <link name="${side}_arm_1">
@@ -66,5 +66,5 @@
             </collision>
         </link>
-        <joint name="${side}_arm_1_${side}_arm_2_joint" type="revolute">
+        <joint name="${side}_arm_1_${side}_arm_2_joint" type="continuous">
             <parent link="${side}_arm_1" />
             <child link="${side}_arm_2" />
@@ -72,5 +72,5 @@
             <axis xyz="0 0 1" />
             <dynamics damping="0.1" friction="0.1" />
-            <limit effort="0.0" lower="-3.1416" upper="3.1416" velocity="1000.0" />
+            <limit effort="0.0" velocity="1000.0" />
         </joint>
         <link name="${side}_arm_3">
@@ -95,5 +95,5 @@
             <axis xyz="0 1 0" />
             <dynamics damping="0.1" friction="0.1" />
-            <limit effort="0.0" lower="-3.1416" upper="3.1416" velocity="1000.0" />
+            <limit effort="0.0" lower="-2.3562" upper="2.3562" velocity="1000.0" />
         </joint>
         <link name="${side}_arm_eef">

Commit message: Add temporal ensembling in BC play script, add joint limits in URDF

File: src/taser/common/model/urdf/taser.urdf (robot description, URDF)
Before this commit: robot taser, 17 links, 16 joints
Joints:
- joint base_link_left_arm_shoulder_joint: limit effort=0.0 velocity=1000.0 -> lower=-3.14159 upper=3.14159 effort=0.0 velocity=1000.0
- joint base_link_right_arm_shoulder_joint: limit effort=0.0 velocity=1000.0 -> lower=-3.14159 upper=3.14159 effort=0.0 velocity=1000.0
- joint left_arm_1_left_arm_2_joint: limit effort=0.0 velocity=1000.0 -> lower=-3.14159 upper=3.14159 effort=0.0 velocity=1000.0
- joint right_arm_1_right_arm_2_joint: limit effort=0.0 velocity=1000.0 -> lower=-3.14159 upper=3.14159 effort=0.0 velocity=1000.0

File: src/taser/common/model/urdf/xacro/arm.xacro (robot description, xacro)
@@ -29,5 +29,5 @@
             <axis xyz="0 1 0" />
             <dynamics damping="0.1" friction="0.1" />
-            <limit effort="0.0" velocity="1000.0" />
+            <limit effort="0.0" velocity="1000.0" lower="-3.14159" upper="3.14159" />
         </joint>
         <link name="${side}_arm_1">
@@ -72,5 +72,5 @@
             <axis xyz="0 0 1" />
             <dynamics damping="0.1" friction="0.1" />
-            <limit effort="0.0" velocity="1000.0" />
+            <limit effort="0.0" velocity="1000.0" lower="-3.14159" upper="3.14159" />
         </joint>
         <link name="${side}_arm_3">
