Commit message: Fix navigation, display path in rviz, update cli, improve logger, add parameter yaml file

File: src/taser_ros/taser_ros/config/taser.urdf (robot description, URDF)
Before this commit: robot taser, 23 links, 22 joints
Links:
- removed link left_arm_shoulder
- removed link left_arm_shoulder_bridge
- removed link right_arm_shoulder
- removed link right_arm_shoulder_bridge
- added link left_arm_6; collision box size=0.05 0.1 0.05; visual box size=0.05 0.1 0.05
- added link left_arm_gripper1; collision box size=0.05 0.0125 0.1; visual box size=0.05 0.0125 0.1
- added link left_arm_gripper2; collision box size=0.05 0.0125 0.1; visual box size=0.05 0.0125 0.1
- added link right_arm_6; collision box size=0.05 0.1 0.05; visual box size=0.05 0.1 0.05
- added link right_arm_gripper1; collision box size=0.05 0.0125 0.1; visual box size=0.05 0.0125 0.1
- added link right_arm_gripper2; collision box size=0.05 0.0125 0.1; visual box size=0.05 0.0125 0.1
- link left_arm_1: geometry collision cylinder length=0.05 radius=0.075; visual cylinder length=0.05 radius=0.075
- link left_arm_2: geometry collision box size=0.1 0.1 0.2; visual box size=0.1 0.1 0.2
- link left_arm_3: geometry collision box size=0.05 0.05 0.15; visual box size=0.05 0.05 0.15
- link left_arm_4: geometry collision box size=0.05 0.05 0.15; visual box size=0.05 0.05 0.15
- link left_arm_5: geometry collision box size=0.05 0.05 0.15; visual box size=0.05 0.05 0.15
- link right_arm_1: geometry collision cylinder length=0.05 radius=0.075; visual cylinder length=0.05 radius=0.075
- link right_arm_2: geometry collision box size=0.1 0.1 0.2; visual box size=0.1 0.1 0.2
- link right_arm_3: geometry collision box size=0.05 0.05 0.15; visual box size=0.05 0.05 0.15
- link right_arm_4: geometry collision box size=0.05 0.05 0.15; visual box size=0.05 0.05 0.15
- link right_arm_5: geometry collision box size=0.05 0.05 0.15; visual box size=0.05 0.05 0.15
Joints:
- removed joint base_link_left_arm_shoulder_bridge_joint
- removed joint base_link_right_arm_shoulder_bridge_joint
- removed joint left_arm_5_left_arm_eef_joint
- removed joint left_arm_shoulder_bridge_left_arm_shoulder_joint
- removed joint left_arm_shoulder_left_arm_1_joint
- removed joint right_arm_5_right_arm_eef_joint
- removed joint right_arm_shoulder_bridge_right_arm_shoulder_joint
- removed joint right_arm_shoulder_right_arm_1_joint
- added joint base_link_left_arm_1_joint: type revolute, parent base_link, child left_arm_1, origin xyz=0.0 +0.25 0.5 rpy=0.0 0.0 0.0, axis 1 0 0, limit lower=0.0 upper=1.57 effort=0.0 velocity=1000.0
- added joint base_link_right_arm_1_joint: type revolute, parent base_link, child right_arm_1, origin xyz=0.0 -0.25 0.5 rpy=0.0 0.0 0.0, axis 1 0 0, limit lower=-1.57 upper=0.0 effort=0.0 velocity=1000.0
- added joint left_arm_5_left_arm_6_joint: type continuous, parent left_arm_5, child left_arm_6, origin xyz=0.0 0 -0.15 rpy=0.0 0.0 0.0, axis 0 0 1, limit lower=-3.14 upper=3.14 effort=0.0 velocity=1000.0
- added joint left_arm_6_left_arm_eef_joint: type fixed, parent left_arm_6, child left_arm_eef, origin xyz=0.0 0 -0.1 rpy=0.0 0.0 0.0
- added joint left_arm_6_left_arm_gripper1_joint: type prismatic, parent left_arm_6, child left_arm_gripper1, origin xyz=0.0 0.037500000000000006 -0.05 rpy=0.0 0.0 0.0, axis 0 1 0, limit lower=-0.037500000000000006 upper=0.0 effort=0.0 velocity=1000.0
- added joint left_arm_6_left_arm_gripper2_joint: type prismatic, parent left_arm_6, child left_arm_gripper2, origin xyz=0.0 -0.037500000000000006 -0.05 rpy=0.0 0.0 0.0, axis 0 1 0, limit lower=0.0 upper=0.037500000000000006 effort=0.0 velocity=1000.0
- added joint right_arm_5_right_arm_6_joint: type continuous, parent right_arm_5, child right_arm_6, origin xyz=0.0 0 -0.15 rpy=0.0 0.0 0.0, axis 0 0 1, limit lower=-3.14 upper=3.14 effort=0.0 velocity=1000.0
- added joint right_arm_6_right_arm_eef_joint: type fixed, parent right_arm_6, child right_arm_eef, origin xyz=0.0 0 -0.1 rpy=0.0 0.0 0.0
- added joint right_arm_6_right_arm_gripper1_joint: type prismatic, parent right_arm_6, child right_arm_gripper1, origin xyz=0.0 0.037500000000000006 -0.05 rpy=0.0 0.0 0.0, axis 0 1 0, limit lower=-0.037500000000000006 upper=0.0 effort=0.0 velocity=1000.0
- added joint right_arm_6_right_arm_gripper2_joint: type prismatic, parent right_arm_6, child right_arm_gripper2, origin xyz=0.0 -0.037500000000000006 -0.05 rpy=0.0 0.0 0.0, axis 0 1 0, limit lower=0.0 upper=0.037500000000000006 effort=0.0 velocity=1000.0
- joint left_arm_1_left_arm_2_joint: limit effort=0.0 velocity=1000.0 -> lower=-3.14 upper=3.14 effort=0.0 velocity=1000.0; origin xyz=0.0 0 -0.1 rpy=0.0 0.0 0.0 -> xyz=0.0 +0.075 0.0 rpy=0.0 0.0 0.0
- joint left_arm_2_left_arm_3_joint: axis 1 0 0 -> 0 0 1; limit effort=0.0 velocity=1000.0 -> lower=-3.14 upper=3.14 effort=0.0 velocity=1000.0
- joint left_arm_3_left_arm_4_joint: axis 0 0 1 -> 0 1 0; limit effort=0.0 velocity=1000.0 -> lower=-3.14 upper=3.14 effort=0.0 velocity=1000.0; origin xyz=0.0 0 -0.1 rpy=0.0 0.0 0.0 -> xyz=0.0 0 -0.15 rpy=0.0 0.0 0.0
- joint left_arm_4_left_arm_5_joint: limit lower=-2.3562 upper=2.3562 effort=0.0 velocity=1000.0 -> lower=-3.14 upper=3.14 effort=0.0 velocity=1000.0; origin xyz=0.0 0 -0.1 rpy=0.0 0.0 0.0 -> xyz=0.0 0 -0.15 rpy=0.0 0.0 0.0
- joint right_arm_1_right_arm_2_joint: limit effort=0.0 velocity=1000.0 -> lower=-3.14 upper=3.14 effort=0.0 velocity=1000.0; origin xyz=0.0 0 -0.1 rpy=0.0 0.0 0.0 -> xyz=0.0 -0.075 0.0 rpy=0.0 0.0 0.0
- joint right_arm_2_right_arm_3_joint: axis 1 0 0 -> 0 0 1; limit effort=0.0 velocity=1000.0 -> lower=-3.14 upper=3.14 effort=0.0 velocity=1000.0
- joint right_arm_3_right_arm_4_joint: axis 0 0 1 -> 0 1 0; limit effort=0.0 velocity=1000.0 -> lower=-3.14 upper=3.14 effort=0.0 velocity=1000.0; origin xyz=0.0 0 -0.1 rpy=0.0 0.0 0.0 -> xyz=0.0 0 -0.15 rpy=0.0 0.0 0.0
- joint right_arm_4_right_arm_5_joint: limit lower=-2.3562 upper=2.3562 effort=0.0 velocity=1000.0 -> lower=-3.14 upper=3.14 effort=0.0 velocity=1000.0; origin xyz=0.0 0 -0.1 rpy=0.0 0.0 0.0 -> xyz=0.0 0 -0.15 rpy=0.0 0.0 0.0
